File: test2/_autosave-test2.kicad_pcb (KiCad board)
At the start: 2 copper layers, 100 x 100 mm, 18 parts, among them J1 USB_B_Micro, X1 Badgelife_sao_connector_v169b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

Commit message: .
Parts:
- added REF**: ProtoBoard, test2:ProtoBoard, F.Cu at (91.9, 88.9)
Routing:
- net (no net): track 0.00 -> 145.7 mm
- net Net-(D2-Pad1): track 0.00 -> 28.4 mm
- net Net-(D3-Pad1): track 0.00 -> 26.6 mm
