File: test2/test2.sch (KiCad schematic (older format))
At the start: 5 parts, among them J1 USB_B_Micro, X1 Badgelife_sao_connector_v169b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

Commit message: .
Parts:
- D1, D2, D3: footprint digikey-footprints:LED_2-SMD_Gull_Wing_4.4x3.85mm -> plcc4:MF_LEDs-PLCC4
- X1: symbol badgelife_shitty_addon_v169bis:Badgelife_sao_connector_v169bis -> test2-rescue:Badgelife_sao_connector_v169bis-badgelife_shitty_addon_v169bis
Changed lines of the file:
@@
 EESchema Schematic File Version 4
+LIBS:test2-cache
 EELAYER 30 0
 EELAYER END
@@
 $EndComp
 $Comp
-L badgelife_shitty_addon_v169bis:Badgelife_sao_connector_v169bis X1
+L test2-rescue:Badgelife_sao_connector_v169bis-badgelife_shitty_addon_v169bis X1
 U 1 1 5D5EDCBC
 P 4950 2950
@@
 F 0 "D1" H 2100 4597 50  0000 C CNN
 F 1 "LED_RGBA" H 2100 4506 50  0000 C CNN
-F 2 "digikey-footprints:LED_2-SMD_Gull_Wing_4.4x3.85mm" H 2100 4050 50  0001 C CNN
+F 2 "plcc4:MF_LEDs-PLCC4" H 2100 4050 50  0001 C CNN
 F 3 "~" H 2100 4050 50  0001 C CNN
 	1    2100 4100
@@
 F 0 "D2" H 2800 4597 50  0000 C CNN
 F 1 "LED_RGBA" H 2800 4506 50  0000 C CNN
-F 2 "digikey-footprints:LED_2-SMD_Gull_Wing_4.4x3.85mm" H 2800 4050 50  0001 C CNN
+F 2 "plcc4:MF_LEDs-PLCC4" H 2800 4050 50  0001 C CNN
 F 3 "~" H 2800 4050 50  0001 C CNN
 	1    2800 4100
@@
 F 0 "D3" H 3450 4597 50  0000 C CNN
 F 1 "LED_RGBA" H 3450 4506 50  0000 C CNN
-F 2 "digikey-footprints:LED_2-SMD_Gull_Wing_4.4x3.85mm" H 3450 4050 50  0001 C CNN
+F 2 "plcc4:MF_LEDs-PLCC4" H 3450 4050 50  0001 C CNN
 F 3 "~" H 3450 4050 50  0001 C CNN
 	1    3450 4100
