File: test2/test2.kicad_pcb (KiCad board)
At the start: 2 copper layers, 5 parts, among them J1 USB_B_Micro, X1 Badgelife_sao_connector_v169b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

Commit message: .
Parts:
- added REF**: ProtoBoard, test2:ProtoBoard, F.Cu at (91.9, 88.9)
- added REF**: dot, test2:dot, F.Cu at (130.8, 66.5)
- added REF**: dot, test2:dot, F.Cu at (130.3, 66.5)
- added REF**: dot, test2:dot, F.Cu at (129.8, 66.5)
- added REF**: dot, test2:dot, F.Cu at (129.3, 66.5)
- added REF**: dot, test2:dot, F.Cu at (128.8, 66.5)
- added REF**: DIP-24_W15.24mm, Package_DIP:DIP-24_W15.24mm, F.Cu at (71.6, 92.5)
- added REF**: dot-1mm, test2:dot-1mm, F.Cu at (131.8, 69.1)
- added REF**: dot-1mm, test2:dot-1mm, F.Cu at (130.3, 69.1)
- added REF**: dot-1mm, test2:dot-1mm, F.Cu at (128.8, 69.1)
- added REF**: dot-0.5mm, test2:dot-0.5mm, F.Cu at (131.6, 67.6)
- added REF**: dot-0.5mm, test2:dot-0.5mm, F.Cu at (130.6, 67.6)
- added REF**: dot-0.5mm, test2:dot-0.5mm, F.Cu at (129.5, 67.6)
- added REF**: dot-0.5mm, test2:dot-0.5mm, F.Cu at (128.5, 67.6)
- D1, D2, D3: footprint digikey-footprints:LED_2-SMD_Gull_Wing_4.4x3.85mm -> plcc4:MF_LEDs-PLCC4
- moved D2 92.4 mm to (79.7, 69.4), turned to 180 degrees
- moved X1 85.0 mm to (84.8, 54.6)
- moved D3 76.6 mm to (93.2, 69.8), turned to 180 degrees
- moved D1 60.2 mm to (104.6, 71.1)
- moved J1 52.9 mm to (159.8, 51.1), turned to 90 degrees
Routing:
- net (no net): vias 0 -> 14
Other:
- board outline added: 100 x 100 mm
- board text added: "Arduino Pro Nano"
- board text added: "Back Only"
- board text added: "Front + Back"
- board text added: "Neither"

Commit message: First BOM
Parts:
- added REF**: ssu, test2:ssu, F.Cu at (76.7, 138.4)
- added REF**: ssu, test2:ssu, F.Cu at (155.4, 67.1)
- added REF**: ssu, test2:ssu, F.Cu at (139.4, 53.1)
- added REF**: ssu, test2:ssu, F.Cu at (155.4, 52.8)
- moved J1 87.9 mm to (160.3, 138.9), turned to 0 degrees
- moved X1 85.3 mm to (153.9, 104.6)
- moved REF** 3.95 mm to (74.4, 95.2)
- moved D2 1.32 mm to (105.9, 70.9)
- turned D1 to 0 degrees
- turned D2 to 0 degrees
- renumbered D2 to D1, D1 to D2, D3 to D2
Routing:
- net (no net): track 0.00 -> 739.9 mm, vias 14 -> 15
- net Net-(J1-Pad5): track 0.00 -> 43.7 mm
- net Net-(D2-Pad2): track 0.00 -> 43.1 mm
- net Net-(D2-Pad1): track 0.00 -> 42.6 mm
- net Net-(J1-Pad4): track 0.00 -> 41.3 mm
- net Net-(D2-Pad4): track 0.00 -> 41.1 mm
- net Net-(J1-Pad3): track 0.00 -> 38.9 mm
- net Net-(D3-Pad1): track 0.00 -> 38.5 mm
- net Net-(D3-Pad2): track 0.00 -> 38.3 mm
- net Net-(D2-Pad3): track 0.00 -> 37.4 mm
- net Net-(J1-Pad2): track 0.00 -> 36.9 mm
- net Net-(X1-Pad2): track 0.00 -> 35.3 mm
- net Net-(X1-Pad6): track 0.00 -> 35.1 mm
- net Net-(J1-Pad1): track 0.00 -> 34.5 mm
- net Net-(D3-Pad4): track 0.00 -> 33.2 mm
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Other:
- board text added: "1"
- board text added: "1, 24"
- board text added: "10,15"
- board text added: "11,14"
- board text added: "12,13"
- board text added: "2"
- board text added: "2, 23"
- board text added: "3"
- board text added: "3, 22"
- board text added: "4"
- board text added: "4, 21"
- board text added: "5"
- board text added: "5, 20"
- board text added: "6, 19"
- board text added: "7, 18"
- board text added: "8, 17"
- board text added: "9, 16"
- board text added: "A"
- board text added: "B"
- board text added: "C"
- board text added: "D"
- board text added: "D1"
- board text added: "D2"
- board text added: "D3"
- board text added: "SAO Header"

Commit message: added stuff
Parts:
- added REF**: 10x7_ProtoBoard, test2:10x7_ProtoBoard, F.Cu at (134.1, 74.7)
- added REF**: 20x6 ProtoBoard, test2:20x6 ProtoBoard, F.Cu at (69.6, 45.2)
