File: hello_world/_autosave-hello_world.kicad_pcb (KiCad board)
At the start: 2 copper layers, 99.1 x 76.2 mm, 15 parts, among them Q1 2N3904, U1 7555

Commit message: I guess this is a checkin
Routing:
- net GND: track 108.0 -> 109.9 mm
Changed lines of the file:
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@@
     (thickness 1.6)
     (drawings 9)
-    (tracks 91)
+    (tracks 94)
     (zones 0)
     (modules 15)
@@
     (33 F.Adhes user hide)
     (34 B.Paste user hide)
-    (35 F.Paste user)
+    (35 F.Paste user hide)
     (36 B.SilkS user hide)
-    (37 F.SilkS user)
+    (37 F.SilkS user hide)
     (38 B.Mask user hide)
-    (39 F.Mask user)
+    (39 F.Mask user hide)
     (40 Dwgs.User user hide)
     (41 Cmts.User user hide)
@@
     (45 Margin user hide)
     (46 B.CrtYd user hide)
-    (47 F.CrtYd user)
+    (47 F.CrtYd user hide)
     (48 B.Fab user hide)
-    (49 F.Fab user)
+    (49 F.Fab user hide)
   )
   (setup
@@
   (segment (start 170.688 102.362) (end 174.498 106.172) (width 0.254) (layer B.Cu) (net 1))
   (segment (start 174.498 119.126) (end 176.022 119.126) (width 0.254) (layer B.Cu) (net 1))
-  (segment (start 174.498 110.022) (end 183.348 118.872) (width 0.254) (layer B.Cu) (net 1))
   (segment (start 174.498 106.68) (end 174.498 110.022) (width 0.254) (layer B.Cu) (net 1))
-  (segment (start 174.498 106.68) (end 174.498 119.126) (width 0.254) (layer B.Cu) (net 1))
   (segment (start 174.498 106.172) (end 174.498 106.68) (width 0.254) (layer B.Cu) (net 1))
   (segment (start 161.0614 130.2766) (end 167.9448 130.2766) (width 0.254) (layer F.Cu) (net 1))
@@
   (segment (start 174.498 119.126) (end 174.498 121.412) (width 0.254) (layer F.Cu) (net 1))
   (segment (start 174.498 121.412) (end 167.9448 127.9652) (width 0.254) (layer F.Cu) (net 1))
+  (segment (start 174.498 111.252) (end 179.832 111.252) (width 0.254) (layer B.Cu) (net 1))
+  (segment (start 174.498 111.252) (end 174.498 119.126) (width 0.254) (layer B.Cu) (net 1))
+  (segment (start 174.498 106.68) (end 174.498 111.252) (width 0.254) (layer B.Cu) (net 1))
+  (segment (start 183.348 114.768) (end 183.348 118.872) (width 0.254) (layer B.Cu) (net 1))
+  (segment (start 179.832 111.252) (end 183.348 114.768) (width 0.254) (layer B.Cu) (net 1))
   (segment (start 151.184999 105.181001) (end 150.225401 105.181001) (width 0.254) (layer F.Cu) (net 2))
   (segment (start 156.972 99.394) (end 151.184999 105.181001) (width 0.254) (layer F.Cu) (net 2))
