File: bob_ws2811_driver/bob_ws2811_driver.kicad_pcb (KiCad board)
At the start: 2 copper layers, 100 x 50 mm, 50 parts

Commit message: sizing adjustments
Parts:
- removed the REF** at (183.6, 32.9)
- removed the REF** at (164.7, 28.6)
- removed the REF** at (145.7, 32.9)
- removed the REF** at (149.9, 41.9)
- removed the REF** at (145.7, 41.9)
- removed the REF** at (141.5, 41.9)
- removed the REF** at (145.7, 28.6)
- removed the REF** at (127.9, 32.9)
- removed the REF** at (132.1, 41.9)
- removed the REF** at (127.9, 41.9)
- removed the REF** at (123.7, 41.9)
- removed the REF** at (187.8, 41.9)
- removed the REF** at (127.9, 28.6)
- removed the REF** at (183.9, 64.3)
- removed the REF** at (183.9, 55.2)
- removed the REF** at (188.1, 64.3)
- removed the REF** at (179.7, 64.3)
- removed the REF** at (183.9, 50.9)
- removed the REF** at (164.8, 64.4)
- removed the REF** at (164.8, 55.4)
- removed the REF** at (160.7, 64.4)
- removed the REF** at (169.0, 64.4)
- removed the REF** at (183.6, 41.9)
- removed the REF** at (164.8, 51.1)
- removed the REF** at (150.0, 64.5)
- removed the REF** at (145.8, 64.5)
- removed the REF** at (141.6, 64.5)
- removed the REF** at (145.8, 51.2)
- removed the REF** at (145.8, 55.5)
- removed the REF** at (132.2, 64.6)
- removed the REF** at (128.0, 64.6)
- removed the REF** at (123.8, 64.6)
- removed the REF** at (128.0, 55.6)
- removed the REF** at (179.5, 41.9)
- removed the REF** at (128.0, 51.3)
- removed the REF** at (110.2, 55.8)
- removed the REF** at (114.4, 64.8)
- removed the REF** at (110.2, 64.8)
- removed the REF** at (106.0, 64.8)
- removed the REF** at (110.2, 51.4)
- removed the REF** at (110.2, 32.9)
- removed the REF** at (114.4, 41.9)
- removed the REF** at (110.2, 28.6)
- removed the REF** at (110.2, 41.9)
- removed the REF** at (183.6, 28.6)
- removed the REF** at (106.0, 41.9)
- removed the REF** at (168.9, 41.9)
- removed the REF** at (164.7, 41.9)
- removed the REF** at (160.5, 41.9)
- added REF**: WS2811-Driver-Chip, ShiftyBit:WS2811-Driver-Chip, F.Cu at (111.6, 65.8)
- added REF**: 4x1_ProtoBoard, TEST2:4x1_ProtoBoard, F.Cu at (140.2, 66.2)
- added REF**: 4x1_ProtoBoard, TEST2:4x1_ProtoBoard, F.Cu at (157.5, 56.9)
- added REF**: 4x1_ProtoBoard, TEST2:4x1_ProtoBoard, F.Cu at (151.6, 66.3)
- added REF**: 4x1_ProtoBoard, TEST2:4x1_ProtoBoard, F.Cu at (163.1, 66.3)
- added REF**: WS2811-Driver-Chip, ShiftyBit:WS2811-Driver-Chip, F.Cu at (157.5, 66.0)
- added REF**: VAL**, ShiftyBit:SunLed, B.Cu at (157.5, 52.5)
- added REF**: 4x1_ProtoBoard, TEST2:4x1_ProtoBoard, F.Cu at (185.9, 66.4)
- added REF**: VAL**, ShiftyBit:SunLed, B.Cu at (180.3, 52.6)
- added REF**: 4x1_ProtoBoard, TEST2:4x1_ProtoBoard, F.Cu at (174.5, 66.4)
- added REF**: 4x1_ProtoBoard, TEST2:4x1_ProtoBoard, F.Cu at (180.3, 57.0)
- added REF**: VAL**, ShiftyBit:SunLed, B.Cu at (111.6, 52.2)
- added REF**: WS2811-Driver-Chip, ShiftyBit:WS2811-Driver-Chip, F.Cu at (180.3, 66.2)
- added REF**: 4x1_ProtoBoard, TEST2:4x1_ProtoBoard, F.Cu at (186.1, 42.4)
- added REF**: VAL**, ShiftyBit:SunLed, B.Cu at (180.5, 28.6)
- added REF**: 4x1_ProtoBoard, TEST2:4x1_ProtoBoard, F.Cu at (180.5, 33.0)
- added REF**: 4x1_ProtoBoard, TEST2:4x1_ProtoBoard, F.Cu at (174.6, 42.4)
- added REF**: WS2811-Driver-Chip, ShiftyBit:WS2811-Driver-Chip, F.Cu at (180.5, 42.2)
- added REF**: 4x1_ProtoBoard, TEST2:4x1_ProtoBoard, F.Cu at (157.7, 33.0)
- added REF**: WS2811-Driver-Chip, ShiftyBit:WS2811-Driver-Chip, F.Cu at (157.7, 42.2)
- added REF**: VAL**, ShiftyBit:SunLed, B.Cu at (157.7, 28.6)
- added REF**: 4x1_ProtoBoard, TEST2:4x1_ProtoBoard, F.Cu at (151.9, 42.4)
- added REF**: 4x1_ProtoBoard, TEST2:4x1_ProtoBoard, F.Cu at (111.6, 56.6)
- added REF**: 4x1_ProtoBoard, TEST2:4x1_ProtoBoard, F.Cu at (163.3, 42.4)
- added REF**: VAL**, ShiftyBit:SunLed, B.Cu at (134.9, 28.6)
- added REF**: 4x1_ProtoBoard, TEST2:4x1_ProtoBoard, F.Cu at (129.0, 42.4)
- added REF**: 4x1_ProtoBoard, TEST2:4x1_ProtoBoard, F.Cu at (140.5, 42.4)
- added REF**: WS2811-Driver-Chip, ShiftyBit:WS2811-Driver-Chip, F.Cu at (134.9, 42.2)
- added REF**: 4x1_ProtoBoard, TEST2:4x1_ProtoBoard, F.Cu at (134.9, 33.0)
- added REF**: 4x1_ProtoBoard, TEST2:4x1_ProtoBoard, F.Cu at (117.5, 42.4)
- added REF**: 4x1_ProtoBoard, TEST2:4x1_ProtoBoard, F.Cu at (106.0, 42.4)
- added REF**: WS2811-Driver-Chip, ShiftyBit:WS2811-Driver-Chip, F.Cu at (111.9, 42.2)
- added REF**: VAL**, ShiftyBit:SunLed, B.Cu at (111.9, 28.6)
- added REF**: 4x1_ProtoBoard, TEST2:4x1_ProtoBoard, F.Cu at (105.8, 66.0)
- added REF**: 4x1_ProtoBoard, TEST2:4x1_ProtoBoard, F.Cu at (117.2, 66.0)
- added REF**: WS2811-Driver-Chip, ShiftyBit:WS2811-Driver-Chip, F.Cu at (134.6, 65.9)
- added REF**: VAL**, ShiftyBit:SunLed, B.Cu at (134.6, 52.3)
- added REF**: 4x1_ProtoBoard, TEST2:4x1_ProtoBoard, F.Cu at (134.6, 56.8)
- added REF**: 4x1_ProtoBoard, TEST2:4x1_ProtoBoard, F.Cu at (128.8, 66.2)
- moved REF** 52.8 mm to (111.9, 33.0)
Routing:
- net (no net): track 499.0 -> 171.1 mm
Other:
- board text added: "Icarus v2.1"
- board text removed: "Icarus v2.0"
